File: SmartSpeaker/ClearSound.kicad_sch (KiCad schematic)
At the start: 51 parts

Commit message: Programmer UART header
Parts:
- removed L?: 10µH, symbol Device:L_Iron
- added L?: (no value), symbol Device:L_Iron
Connections:
- net at C?.2, IC?.18 (OUTPR), IC?.20 (OUTNR): now also L?.1
- net at C?.1: now also L?.2
Other:
- moved on the sheet: J?
Changed lines of the file:
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@@
     (stroke (width 0) (type default) (color 0 0 0 0))
   )
+  (polyline (pts (xy 12.7 135.89) (xy 142.24 135.89))
+    (stroke (width 0) (type default) (color 0 0 0 0))
+  )
   (wire (pts (xy 491.49 144.78) (xy 491.49 151.13))
     (stroke (width 0) (type default) (color 0 0 0 0))
@@
     (stroke (width 0) (type default) (color 0 0 0 0))
   )
+  (polyline (pts (xy 140.97 12.7) (xy 142.24 12.7))
+    (stroke (width 0) (type default) (color 0 0 0 0))
+  )
   (wire (pts (xy 490.22 266.7) (xy 492.76 266.7))
     (stroke (width 0) (type default) (color 0 0 0 0))
@@
     (stroke (width 0) (type default) (color 0 0 0 0))
   )
+  (polyline (pts (xy 142.24 135.89) (xy 142.24 12.7))
+    (stroke (width 0) (type default) (color 0 0 0 0))
+  )
   (wire (pts (xy 528.32 242.57) (xy 543.56 242.57))
     (stroke (width 0) (type default) (color 0 0 0 0))
@@
     (stroke (width 0) (type default) (color 0 0 0 0))
   )
+  (label "programmer" (at 27.94 35.56 0)
+    (effects (font (size 8 8)) (justify left bottom))
+  )
   (global_label "AVCC" (shape input) (at 508 134.62 0) (fields_autoplaced)
     (effects (font (size 1.27 1.27)) (justify left))
@@
     (pin "1")
   )
-  (symbol (lib_id "Connector:Conn_01x10_Male") (at 44.45 496.57 0) (unit 1)
+  (symbol (lib_id "Connector:Conn_01x10_Male") (at 31.75 69.85 0) (unit 1)
     (in_bom yes) (on_board yes) (fields_autoplaced)
-    (property "Reference" "J?" (id 0) (at 45.085 481.33 0))
-    (property "Value" "UART_DSP" (id 1) (at 45.085 483.87 0))
-    (property "Footprint" "" (id 2) (at 44.45 496.57 0)
+    (property "Reference" "J?" (id 0) (at 32.385 54.61 0))
+    (property "Value" "UART_DSP" (id 1) (at 32.385 57.15 0))
+    (property "Footprint" "" (id 2) (at 31.75 69.85 0)
       (effects (font (size 1.27 1.27)) hide)
     )
-    (property "Datasheet" "~" (id 3) (at 44.45 496.57 0)
+    (property "Datasheet" "~" (id 3) (at 31.75 69.85 0)
       (effects (font (size 1.27 1.27)) hide)
     )
@@
     (pin "2")
   )
-  (symbol (lib_id "Connector:Conn_01x10_Male") (at 44.45 535.94 0) (unit 1)
+  (symbol (lib_id "Connector:Conn_01x10_Male") (at 31.75 109.22 0) (unit 1)
     (in_bom yes) (on_board yes) (fields_autoplaced)
-    (property "Reference" "J?" (id 0) (at 45.085 520.7 0))
-    (property "Value" "UART_WI-FI" (id 1) (at 45.085 523.24 0))
-    (property "Footprint" "" (id 2) (at 44.45 535.94 0)
+    (property "Reference" "J?" (id 0) (at 32.385 93.98 0))
+    (property "Value" "UART_WI-FI" (id 1) (at 32.385 96.52 0))
+    (property "Footprint" "" (id 2) (at 31.75 109.22 0)
       (effects (font (size 1.27 1.27)) hide)
     )
-    (property "Datasheet" "~" (id 3) (at 44.45 535.94 0)
+    (property "Datasheet" "~" (id 3) (at 31.75 109.22 0)
       (effects (font (size 1.27 1.27)) hide)
     )
@@
     (in_bom yes) (on_board yes) (fields_autoplaced)
     (property "Reference" "L?" (id 0) (at 516.89 254 90))
-    (property "Value" "10µH" (id 1) (at 516.89 256.54 90))
+    (property "Value" "" (id 1) (at 516.89 256.54 90))
     (property "Footprint" "" (id 2) (at 516.89 260.35 0)
       (effects (font (size 1.27 1.27)) hide)
@@
       (reference "L?") (unit 1) (value "10µH") (footprint "")
     )
-    (path "/e0ab7642-a04d-4587-90cd-89269620b705"
+    (path "/e0ab7642-a04d-4587-90cd-89269620b706"
       (reference "L?") (unit 1) (value "10µH") (footprint "")
     )

Commit message: UART connections wi-fi chip
Parts:
- L?: value (none) -> 10µH
Connections:
- net WIFI UART TX: now reaches IC?.L9 (UART_TXD)
- net WIFI UART RX: now reaches IC?.M10 (UART_RXD)
Changed lines of the file:
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@@
+    (stroke (width 0) (type default) (color 0 0 0 0))
+  )
+  (wire (pts (xy 116.84 713.74) (xy 129.54 713.74))
     (stroke (width 0) (type default) (color 0 0 0 0))
   )
@@
   )
   (polyline (pts (xy 140.97 12.7) (xy 142.24 12.7))
+    (stroke (width 0) (type default) (color 0 0 0 0))
+  )
+  (wire (pts (xy 116.84 698.5) (xy 129.54 698.5))
     (stroke (width 0) (type default) (color 0 0 0 0))
   )
@@
     (effects (font (size 1.27 1.27)) (justify left))
     (property "Intersheet References" "${INTERSHEET_REFS}" (id 0) (at 515.1302 134.5406 0)
+      (effects (font (size 1.27 1.27)) (justify left) hide)
+    )
+  )
+  (global_label "WIFI UART TX" (shape input) (at 129.54 698.5 0) (fields_autoplaced)
+    (effects (font (size 1.27 1.27)) (justify left))
+    (property "Intersheet References" "${INTERSHEET_REFS}" (id 0) (at 144.4717 698.4206 0)
       (effects (font (size 1.27 1.27)) (justify left) hide)
     )
@@
     (property "Intersheet References" "${INTERSHEET_REFS}" (id 0) (at 564.3686 337.895 0)
       (effects (font (size 1.2 1.2)) (justify left) hide)
+    )
+  )
+  (global_label "WIFI UART RX" (shape input) (at 129.54 713.74 0) (fields_autoplaced)
+    (effects (font (size 1.27 1.27)) (justify left))
+    (property "Intersheet References" "${INTERSHEET_REFS}" (id 0) (at 144.7741 713.6606 0)
+      (effects (font (size 1.27 1.27)) (justify left) hide)
     )
   )
@@
     (in_bom yes) (on_board yes) (fields_autoplaced)
     (property "Reference" "L?" (id 0) (at 516.89 254 90))
-    (property "Value" "" (id 1) (at 516.89 256.54 90))
+    (property "Value" "10µH" (id 1) (at 516.89 256.54 90))
     (property "Footprint" "" (id 2) (at 516.89 260.35 0)
       (effects (font (size 1.27 1.27)) hide)
