File: SensorArray/SensorArray/SensorArray.kicad_sch (KiCad schematic)
At the start: 8 parts

Commit message: add ir sensor
Parts:
- added A?: (no value), symbol IR Sensor:MLX90640ESF-BAA-000-TU
- IC?: value (none) -> EKMC7610113K; footprint (none) -> EKMC7610111K
- Q?: value (none) -> 2N3904; footprint (none) -> Package_TO_SOT_THT:TO-92_Inline
- R?: value (none) -> R_Small
- RV?: value (none) -> R_Potentiometer
- U?: value (none) -> ESP8266EX; footprint (none) -> Package_DFN_QFN:QFN-32-1EP_5x5mm_P0.5mm_EP3.45x3.45mm
Changed lines of the file:
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@@
     )
+  )
+  (symbol (lib_id "IR Sensor:MLX90640ESF-BAA-000-TU") (at 168.91 129.54 0) (unit 1)
+    (in_bom yes) (on_board yes) (fields_autoplaced)
+    (property "Reference" "A?" (id 0) (at 168.91 119.38 0))
+    (property "Value" "" (id 1) (at 168.91 121.92 0))
+    (property "Footprint" "" (id 2) (at 168.91 129.54 0)
+      (effects (font (size 1.27 1.27)) (justify left bottom) hide)
+    )
+    (property "Datasheet" "" (id 3) (at 168.91 129.54 0)
+      (effects (font (size 1.27 1.27)) (justify left bottom) hide)
+    )
+    (property "PARTREV" "11" (id 4) (at 168.91 129.54 0)
+      (effects (font (size 1.27 1.27)) (justify left bottom) hide)
+    )
+    (property "MAXIMUM_PACKAGE_HEIGHT" "6.0 mm" (id 5) (at 168.91 129.54 0)
+      (effects (font (size 1.27 1.27)) (justify left bottom) hide)
+    )
+    (property "STANDARD" "IPC-7351B" (id 6) (at 168.91 129.54 0)
+      (effects (font (size 1.27 1.27)) (justify left bottom) hide)
+    )
+    (property "MANUFACTURER" "Melexis" (id 7) (at 168.91 129.54 0)
+      (effects (font (size 1.27 1.27)) (justify left bottom) hide)
+    )
+    (pin "1")
+    (pin "2")
+    (pin "3")
+    (pin "4")
   )
   (symbol (lib_id "MCU_Espressif:ESP8266EX") (at 215.9 72.39 0) (unit 1)
@@
       (effects (font (size 1.27 1.27)) (justify left))
     )
-    (property "Value" "" (id 1) (at 217.9194 102.87 0)
-      (effects (font (size 1.27 1.27)) (justify left))
-    )
-    (property "Footprint" "" (id 2) (at 215.9 105.41 0)
+    (property "Value" "ESP8266EX" (id 1) (at 217.9194 102.87 0)
+      (effects (font (size 1.27 1.27)) (justify left))
+    )
+    (property "Footprint" "Package_DFN_QFN:QFN-32-1EP_5x5mm_P0.5mm_EP3.45x3.45mm" (id 2) (at 215.9 105.41 0)
       (effects (font (size 1.27 1.27)) hide)
     )
@@
       (effects (font (size 1.27 1.27)) (justify left))
     )
-    (property "Value" "" (id 1) (at 96.52 175.2599 0)
-      (effects (font (size 1.27 1.27)) (justify left))
-    )
-    (property "Footprint" "" (id 2) (at 96.52 175.895 0)
+    (property "Value" "2N3904" (id 1) (at 96.52 175.2599 0)
+      (effects (font (size 1.27 1.27)) (justify left))
+    )
+    (property "Footprint" "Package_TO_SOT_THT:TO-92_Inline" (id 2) (at 96.52 175.895 0)
       (effects (font (size 1.27 1.27) italic) (justify left) hide)
     )
@@
       (effects (font (size 1.27 1.27)) hide)
     )
-    (property "Value" "" (id 1) (at 90.17 137.16 0))
+    (property "Value" "VDD" (id 1) (at 90.17 137.16 0))
     (property "Footprint" "" (id 2) (at 90.17 142.24 0)
       (effects (font (size 1.27 1.27)) hide)
@@
       (effects (font (size 1.27 1.27)) (justify right))
     )
-    (property "Value" "" (id 1) (at 96.52 152.3999 0)
+    (property "Value" "R_Potentiometer" (id 1) (at 96.52 152.3999 0)
       (effects (font (size 1.27 1.27)) (justify right))
     )
@@
       (effects (font (size 1.27 1.27)) hide)
     )
-    (property "Value" "" (id 1) (at 19.05 162.56 0))
+    (property "Value" "GND" (id 1) (at 19.05 162.56 0))
     (property "Footprint" "" (id 2) (at 19.05 167.64 0)
       (effects (font (size 1.27 1.27)) hide)
@@
       (effects (font (size 1.27 1.27)) (justify left))
     )
-    (property "Value" "" (id 1) (at 96.52 163.8299 0)
+    (property "Value" "R_Small" (id 1) (at 96.52 163.8299 0)
       (effects (font (size 1.27 1.27)) (justify left))
     )
@@
       (effects (font (size 1.27 1.27)) hide)
     )
-    (property "Value" "" (id 1) (at 105.41 191.77 0))
+    (property "Value" "GND" (id 1) (at 105.41 191.77 0))
     (property "Footprint" "" (id 2) (at 105.41 186.69 0)
       (effects (font (size 1.27 1.27)) hide)
@@
     (in_bom yes) (on_board yes) (fields_autoplaced)
     (property "Reference" "IC?" (id 0) (at 48.26 181.61 0))
-    (property "Value" "" (id 1) (at 48.26 179.07 0))
-    (property "Footprint" "" (id 2) (at 39.37 176.53 0)
+    (property "Value" "EKMC7610113K" (id 1) (at 48.26 179.07 0))
+    (property "Footprint" "EKMC7610111K" (id 2) (at 39.37 176.53 0)
       (effects (font (size 1.27 1.27)) (justify left) hide)
     )
@@
       (reference "#PWR?") (unit 1) (value "GND") (footprint "")
     )
+    (path "/078063ad-497c-4f95-b99c-ef390ce3bc98"
+      (reference "A?") (unit 1) (value "MLX90640ESF-BAA-000-TU") (footprint "TO292P930H600-4")
+    )
     (path "/ca4c5752-be14-45f9-9713-c386613e0fce"

Commit message: add ir sensor
Parts:
- A?: value (none) -> MLX90640ESF-BAA-000-TU; footprint (none) -> TO292P930H600-4
Changed lines of the file:
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@@
     (in_bom yes) (on_board yes) (fields_autoplaced)
     (property "Reference" "A?" (id 0) (at 168.91 119.38 0))
-    (property "Value" "" (id 1) (at 168.91 121.92 0))
-    (property "Footprint" "" (id 2) (at 168.91 129.54 0)
+    (property "Value" "MLX90640ESF-BAA-000-TU" (id 1) (at 168.91 121.92 0))
+    (property "Footprint" "TO292P930H600-4" (id 2) (at 168.91 129.54 0)
       (effects (font (size 1.27 1.27)) (justify left bottom) hide)
     )
