File: SensorArray/SensorArray/SensorArray.kicad_sch (KiCad schematic)
At the start: 1 part

Commit message: Dongbin
Parts:
- added IC?: (no value), symbol Mt Sensor:EKMC7610113K
- added Q?: (no value), symbol Transistor_BJT:2N3904
- added R? (x2): R_Small, symbol Device:R_Small
- added R?: (no value), symbol Device:R_Small
- added RV?: (no value), symbol Device:R_Potentiometer
- added U?: (no value), symbol MCU_Espressif:ESP8266EX
- U?: value (none) -> R7FS128783A01CFJ-AA1; footprint (none) -> PLQP0032GB-A_REN
Connections:
- net VDD: now reaches U?.7 (VCC)
- net VDD: now also IC?.1 (VDD), RV?.2
- new net: Q?.2 (B), R?.1, R?.2
- new net: Q?.3 (C), R?.2
- new net: R?.1, RV?.1
- new net: IC?.2 (OUT), R?.2
- new net GND: IC?.3 (GND), Q?.1 (E), R?.1
- no-connect marks 0 -> 1
Other:
- moved on the sheet: U?

Commit message: changes
Parts:
- IC?: value (none) -> EKMC7610113K; footprint (none) -> EKMC7610111K
- Q?: value (none) -> 2N3904; footprint (none) -> Package_TO_SOT_THT:TO-92_Inline
- R?: value (none) -> R_Small
- RV?: value (none) -> R_Potentiometer
- U?: value (none) -> ESP8266EX; footprint (none) -> Package_DFN_QFN:QFN-32-1EP_5x5mm_P0.5mm_EP3.45x3.45mm
Changed lines of the file:
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@@
       (effects (font (size 1.27 1.27)) (justify left))
     )
-    (property "Value" "" (id 1) (at 217.9194 102.87 0)
-      (effects (font (size 1.27 1.27)) (justify left))
-    )
-    (property "Footprint" "" (id 2) (at 215.9 105.41 0)
+    (property "Value" "ESP8266EX" (id 1) (at 217.9194 102.87 0)
+      (effects (font (size 1.27 1.27)) (justify left))
+    )
+    (property "Footprint" "Package_DFN_QFN:QFN-32-1EP_5x5mm_P0.5mm_EP3.45x3.45mm" (id 2) (at 215.9 105.41 0)
       (effects (font (size 1.27 1.27)) hide)
     )
@@
       (effects (font (size 1.27 1.27)) (justify left))
     )
-    (property "Value" "" (id 1) (at 96.52 175.2599 0)
-      (effects (font (size 1.27 1.27)) (justify left))
-    )
-    (property "Footprint" "" (id 2) (at 96.52 175.895 0)
+    (property "Value" "2N3904" (id 1) (at 96.52 175.2599 0)
+      (effects (font (size 1.27 1.27)) (justify left))
+    )
+    (property "Footprint" "Package_TO_SOT_THT:TO-92_Inline" (id 2) (at 96.52 175.895 0)
       (effects (font (size 1.27 1.27) italic) (justify left) hide)
     )
@@
       (effects (font (size 1.27 1.27)) hide)
     )
-    (property "Value" "" (id 1) (at 90.17 137.16 0))
+    (property "Value" "VDD" (id 1) (at 90.17 137.16 0))
     (property "Footprint" "" (id 2) (at 90.17 142.24 0)
       (effects (font (size 1.27 1.27)) hide)
@@
       (effects (font (size 1.27 1.27)) (justify right))
     )
-    (property "Value" "" (id 1) (at 96.52 152.3999 0)
+    (property "Value" "R_Potentiometer" (id 1) (at 96.52 152.3999 0)
       (effects (font (size 1.27 1.27)) (justify right))
     )
@@
       (effects (font (size 1.27 1.27)) hide)
     )
-    (property "Value" "" (id 1) (at 19.05 162.56 0))
+    (property "Value" "GND" (id 1) (at 19.05 162.56 0))
     (property "Footprint" "" (id 2) (at 19.05 167.64 0)
       (effects (font (size 1.27 1.27)) hide)
@@
       (effects (font (size 1.27 1.27)) (justify left))
     )
-    (property "Value" "" (id 1) (at 96.52 163.8299 0)
+    (property "Value" "R_Small" (id 1) (at 96.52 163.8299 0)
       (effects (font (size 1.27 1.27)) (justify left))
     )
@@
       (effects (font (size 1.27 1.27)) hide)
     )
-    (property "Value" "" (id 1) (at 105.41 191.77 0))
+    (property "Value" "GND" (id 1) (at 105.41 191.77 0))
     (property "Footprint" "" (id 2) (at 105.41 186.69 0)
       (effects (font (size 1.27 1.27)) hide)
@@
     (in_bom yes) (on_board yes) (fields_autoplaced)
     (property "Reference" "IC?" (id 0) (at 48.26 181.61 0))
-    (property "Value" "" (id 1) (at 48.26 179.07 0))
-    (property "Footprint" "" (id 2) (at 39.37 176.53 0)
+    (property "Value" "EKMC7610113K" (id 1) (at 48.26 179.07 0))
+    (property "Footprint" "EKMC7610111K" (id 2) (at 39.37 176.53 0)
       (effects (font (size 1.27 1.27)) (justify left) hide)
     )
