File: SensorArray/SensorArray/SensorArray.kicad_sch (KiCad schematic)
At the start: 25 parts

Commit message: Power filter added with Antena
Parts:
- added C?: 10µF, Capacitor_SMD:C_0402_1005Metric, symbol Device:C_Small
- added C? (x5): 0.1µF, Capacitor_SMD:C_0402_1005Metric, symbol Device:C_Small
- added C? (x4): 0.01µF, Capacitor_SMD:C_0402_1005Metric, symbol Device:C_Small
- added C?: C_Small, Capacitor_SMD:C_0402_1005Metric, symbol Device:C_Small
- added D?: D_Small_Filled, Diode_SMD:D_0805_2012Metric, symbol Device:D_Small_Filled
- added L?: L_Ferrite_Small, Inductor_SMD:L_6.3x6.3_H3, symbol Device:L_Ferrite_Small
- 100kOhm: value (none) -> Rpg
- 10kR: value (none) -> R_Small
- 22µFCout: value (none) -> 3.71Ohm
- 470nH: value (none) -> 7.6mOhm
- 806kOhm: value (none) -> Rfbt
- 91kOhm: value (none) -> Rfbb
- J?: value (none) -> Barrel_Jack
Connections:
- net GND: now also C?.1, C?.1, C?.1, C?.1, C?.1, C?.1, C?.1, C?.1, C?.2, C?.2, C?.2, C?.2, C?.2, C?.2, C?.2, C?.2, C?.2, C?.2, C?.2, D?.2 (A), L?.1
- new net VBAT: C?.1, D?.1 (K)
- new net VDDA: C?.1, C?.1, L?.2
Other:
- note added: "Power Filter"
